File: led_hc501/led_hc501.kicad_pcb (KiCad board)
At the start: 2 copper layers, 50 x 30 mm, 14 parts, among them J1 LED02, J10 Conn_01x03_Pin, J11 BATTERY, J2 Conn_01x01_Pin, J3 Conn_01x01_Pin, J4 BUZZ, J5 LED01, J6 HC-SR501_01, J7 Conn_01x01_Pin, J8 Conn_01x01_Pin, J9 LED03, Q3 IRLZ44N

Commit message: [SCHEMATIC] testing
Parts:
- removed J1: LED02, Connector_JST:JST_XH_B2B-XH-A_1x02_P2.50mm_Vertical
- removed J10: Conn_01x03_Pin, Connector_JST:JST_XH_B3B-XH-A_1x03_P2.50mm_Vertical
- removed J11: BATTERY, Connector_JST:JST_XH_B2B-XH-A_1x02_P2.50mm_Vertical
- removed J2, J3, J7, J8: Conn_01x01_Pin, Connector_PinHeader_2.54mm:PinHeader_1x01_P2.54mm_Vertical
- removed J4: BUZZ, Connector_JST:JST_XH_B2B-XH-A_1x02_P2.50mm_Vertical
- removed J5: LED01, Connector_JST:JST_XH_B2B-XH-A_1x02_P2.50mm_Vertical
- removed J6: HC-SR501_01, Connector_PinHeader_2.54mm:PinHeader_1x03_P2.54mm_Horizontal
- removed J9: LED03, Connector_JST:JST_XH_B2B-XH-A_1x02_P2.50mm_Vertical
- removed Q3: IRLZ44N, Package_TO_SOT_THT:TO-220-3_Vertical
- removed R1: 100k, Resistor_THT:R_Axial_DIN0309_L9.0mm_D3.2mm_P2.54mm_Vertical
- removed R4: 1k, Resistor_THT:R_Axial_DIN0309_L9.0mm_D3.2mm_P2.54mm_Vertical
Routing:
- net Net-(J4-Pin_1): track 63.2 -> 0.00 mm
- net GND: track 54.1 -> 0.00 mm
- net input: track 24.8 -> 0.00 mm
- net Net-(Q3-G): track 21.0 -> 0.00 mm
- net Battery-: track 20.6 -> 0.00 mm
- net Net-(J1-Pin_1): track 19.2 -> 0.00 mm
- net Battery+: track 16.8 -> 0.00 mm
- net Net-(J1-Pin_2): track 11.0 -> 0.00 mm
- removed copper zone on F.Cu, net 9v
Other:
- board outline removed
- board text removed: "5V"
- board text removed: "BUZZ"
- board text removed: "Bat+"
- board text removed: "Bat-"
- board text removed: "GND"
- board text removed: "HC-SR501_02"
- board text removed: "Input"
- board text removed: "LED01"
- board text removed: "LED02"
- board text removed: "LED03"
